File: KiCAD/Capstone.kicad_sch (KiCad schematic)
At the start: 12 parts, among them Q1 IRLZ44N, Q2 IRLZ44N, U1 IR2110

Commit message: Add files via upload
Edited the schematic and uploaded the new PDF
Parts:
- removed D1: 1N914, Diode_THT:D_DO-35_SOD27_P7.62mm_Horizontal, symbol Diode:1N914
- removed L1: L_Coupled, symbol Device:L_Coupled
- removed U1: IR2110, Package_DIP:DIP-14_W7.62mm, symbol Driver_FET:IR2110
- added C3, C5: 100n, symbol Device:C_Small_US
- added D1: 1N5819, Diode_THT:D_DO-41_SOD81_P10.16mm_Horizontal, symbol Diode:1N5819
- added J1: 12VDC, symbol Connector_Generic:Conn_01x02
- added TX_coil: 7.3u, symbol Device:L
- added U1: IR2104, symbol Driver_FET:IR2104
- A1: renamed from A2; value RaspberryPi_Pico_W -> RaspberryPi_Pico_2
- C1: renamed from C2; value C_Small_US -> 10u
- C2: renamed from C3; value C_Small_US -> 10u
- CB: renamed from C1; value C_Small_US -> 4.7u
- C_RES: renamed from C4; value C_Small_US -> 220n
- Q1, Q2: value IRLZ44N -> IRFB4410Z
- R1, R2: value R_US -> 22
Connections:
- net +12V: now also C3.1, C5.1, D1.2 (A), J1.1 (Pin_1), U1.1 (VCC)
- net +3.3V: now also U1.3 (~{SD})
- net GND: now also C3.2, C5.2, J1.2 (Pin_2), U1.4 (COM)
- net at C1.2, C2.1: now also TX_coil.2
- net at CB.2, C_RES.1, Q1.3 (S)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: now also U1.6 (VS)
- net at C_RES.2: now also TX_coil.1
- net at R2.2: now also U1.5 (LO)
- net at CB.1: now also D1.1 (K), U1.8 (VB)
- net at R1.2: now also U1.7 (HO)
- net at A1.1 (GPIO0): now also U1.2 (IN)
- no-connect marks 0 -> 30
Other:
- title: (none) -> Wireless Charger Transmitter
- moved on the sheet: A1, C1, C2, CB, C_RES, Q1, Q2, R1, R2
